Commit message: add the walking robot script

File: otto_description/urdf/otto_gz.xacro (robot description, xacro)
@@ -50,5 +50,5 @@
     <gazebo>
       <!-- gz-sim-joint-state-publisher-system -->
-      <!-- JointStatePublisher : Measures the joints in Gazebo frequently -> sends to /joint_states via the bridge ->
+      <!-- JointStatePublisher: Measures the joints in Gazebo frequently -> sends to /joint_states via the bridge ->
       ROS 2 uses Forward Kinematics to calculate the robot's current physical posture.
        -->
@@ -63,5 +63,5 @@
       <!-- gz_ros2_control listen to the logic (Inverse Kinematics) from ROS2 and translate it to the simulation to move the robot. -->
       <plugin filename="gz_ros2_control-system" name="gz_ros2_control::GazeboSimROS2ControlPlugin">
-        <parameters>$(find otto_description)/config/controllers.yaml</parameters>
+        <parameters>$(find otto_description)/config/controllers.yaml</parameters>    <!-- Load the yaml file to gazebo. -->
       </plugin>
     </gazebo>

File: otto_description/urdf/otto_main.urdf.xacro (robot description, xacro)
@@ -27,15 +27,15 @@
   <!-- ── Include utilities ── -->
   <xacro:include filename="otto_materials.xacro" />
-  <xacro:include filename="otto_gz.gazebo" />
+  <xacro:include filename="otto_gz.xacro" />
   <!--==== PHYSICAL PARAMETERS ====-->
   <!-- Body / head combined box -->
   <xacro:property name="body_x"    value="0.075"/>   <!-- width  -->
   <xacro:property name="body_y"    value="0.060"/>   <!-- depth  -->
-  <xacro:property name="body_z"    value="0.080"/>   <!-- height -->
+  <xacro:property name="body_z"    value="0.065"/>   <!-- height -->
   <xacro:property name="body_mass" value="0.120"/>
   <!-- Leg segment -->
   <xacro:property name="leg_x"    value="0.020"/>
   <xacro:property name="leg_y"    value="0.015"/>
-  <xacro:property name="leg_z"    value="0.045"/>
+  <xacro:property name="leg_z"    value="0.035"/>
   <xacro:property name="leg_mass" value="0.025"/>
   <!-- Foot (flat disc) -->
@@ -43,6 +43,6 @@
   <xacro:property name="foot_h"    value="0.008"/>
   <xacro:property name="foot_mass" value="0.020"/>
-  <!-- Servo joint limits (±30° realistic for Otto walk) -->
-  <xacro:property name="servo_limit" value="0.5236"/>   <!-- rad, ~30° -->
+  <!-- Servo joint limits (±40° realistic for Otto walk) -->
+  <xacro:property name="servo_limit" value="0.78"/>   <!-- rad, ~40° -->
   <xacro:property name="servo_vel"   value="3.14"/>     <!-- rad/s     -->
   <xacro:property name="servo_eff"   value="0.5"/>      <!-- N·m       -->
@@ -113,5 +113,5 @@
     <child  link="left_leg_link"/>
     <origin xyz="0 0 ${-leg_z/2.0}" rpy="0 0 0"/>
-    <axis   xyz="0 0 1"/>
+    <axis   xyz="1 0 0"/>
     <limit  lower="${-servo_limit}" upper="${servo_limit}"
             effort="${servo_eff}"   velocity="${servo_vel}"/>
@@ -170,5 +170,5 @@
     <child  link="right_leg_link"/>
     <origin xyz="0 0 ${-leg_z/2.0}" rpy="0 0 0"/>
-    <axis   xyz="0 0 1"/>
+    <axis   xyz="1 0 0"/>
     <limit  lower="${-servo_limit}" upper="${servo_limit}"
             effort="${servo_eff}"   velocity="${servo_vel}"/>

File: otto_description/urdf/otto_materials.xacro (robot description, xacro)
@@ -72,9 +72,9 @@
     <!-- Servo body -->
     <link name="${prefix}_servo">
-      <xacro:inertia_box m="0.009" x="0.023" y="0.012" z="0.032"/>
+      <xacro:inertia_box m="0.009" x="0.023" y="0.012" z="0.045"/>
       <visual>
         <origin xyz="0 0 0" rpy="0 0 0"/>
         <geometry>
-          <box size="0.023 0.012 0.032"/>
+          <box size="0.023 0.012 0.045"/>
         </geometry>
         <material name="otto_dark_grey"/>
@@ -83,5 +83,5 @@
         <origin xyz="0 0 0" rpy="0 0 0"/>
         <geometry>
-          <box size="0.023 0.012 0.032"/>
+          <box size="0.023 0.012 0.045"/>
         </geometry>
       </collision>

Commit message: modified: add rolling ctrl (not working)

File: otto_description/urdf/otto_gz.xacro (robot description, xacro)
@@ -78,4 +78,5 @@
       <joint name="left_foot_joint">
         <command_interface name="position"/>
+        <command_interface name="velocity"/>
         <state_interface name="position"/>
         <state_interface name="velocity"/>
@@ -88,4 +89,5 @@
       <joint name="right_foot_joint">
         <command_interface name="position"/>
+        <command_interface name="velocity"/>
         <state_interface name="position"/>
         <state_interface name="velocity"/>

File: otto_description/urdf/otto_main.urdf.xacro (robot description, xacro)
@@ -210,13 +210,11 @@
     </collision>
   </link>
-  <!-- Foot revolute joint — rotates about Z (tilt foot) -->
-  <joint name="left_foot_joint" type="revolute">
+  <!-- Foot continous joint — rotates about Z (tilt foot) -->
+  <joint name="left_foot_joint" type="continuous">
     <parent link="left_leg_link"/>
     <child  link="left_foot_link"/>
     <origin xyz="0 0 ${foot_z_in_leg - foot_h/2.0}" rpy="0 0 0"/>
     <axis   xyz="0 0 1"/>
-    <limit  lower="${-servo_limit/2}" upper="${servo_limit/2}"
-            effort="${servo_eff}"   velocity="${servo_vel}"/>
-    <xacro:servo_dynamics/>
+    <limit effort="${servo_eff}" velocity="${servo_vel}"/>
   </joint>
   <link name="left_foot_link">
@@ -332,11 +330,10 @@
     </collision>
   </link>
-  <joint name="right_foot_joint" type="revolute">
+  <joint name="right_foot_joint" type="continuous">
     <parent link="right_leg_link"/>
     <child  link="right_foot_link"/>
     <origin xyz="0 0 ${foot_z_in_leg - foot_h/2.0}" rpy="0 0 0"/>
     <axis   xyz="0 0 1"/>
-    <limit  lower="${-servo_limit/2}" upper="${servo_limit/2}"
-            effort="${servo_eff}"   velocity="${servo_vel}"/>
+    <limit effort="${servo_eff}" velocity="${servo_vel}"/>
     <xacro:servo_dynamics/>
   </joint>

Commit message: add rolling...

File: otto_description/urdf/otto_gz.xacro (robot description, xacro)
@@ -78,4 +78,5 @@
       <joint name="left_foot_joint">
         <command_interface name="position"/>
+        <command_interface name="velocity"/>
         <state_interface name="position"/>
         <state_interface name="velocity"/>
@@ -83,4 +84,5 @@
       <joint name="right_hip_joint">
         <command_interface name="position"/>
+        <command_interface name="velocity"/>
         <state_interface name="position"/>
         <state_interface name="velocity"/>

File: otto_description/urdf/otto_main.urdf.xacro (robot description, xacro)
@@ -135,5 +135,5 @@
   </link>
   <!-- Foot revolute joint — rotates about Z (tilt foot) -->
-  <joint name="left_foot_joint" type="revolute">
+  <joint name="left_foot_joint" type="continuous">
     <parent link="left_leg_link"/>
     <child  link="left_foot_link"/>
@@ -191,5 +191,5 @@
     </collision>
   </link>
-  <joint name="right_foot_joint" type="revolute">
+  <joint name="right_foot_joint" type="continuous">
     <parent link="right_leg_link"/>
     <child  link="right_foot_link"/>

Commit message: Restart from gazebo begining

File: otto_description/urdf/otto_gz.xacro (robot description, xacro)
@@ -60,35 +60,4 @@
         <joint_name>right_foot_joint</joint_name>
       </plugin>
-      <!-- gz_ros2_control -->
-      <!-- gz_ros2_control listen to the logic (Inverse Kinematics) from ROS2 and translate it to the simulation to move the robot. -->
-      <plugin filename="gz_ros2_control-system" name="gz_ros2_control::GazeboSimROS2ControlPlugin">
-        <parameters>$(find otto_description)/config/controllers.yaml</parameters>    <!-- Load the yaml file to gazebo. -->
-      </plugin>
     </gazebo>
-    <!-- ROS2_control Specifications -->
-    <ros2_control name="GazeboSimSystem" type="system">
-      <hardware>
-        <plugin>gz_ros2_control/GazeboSimSystem</plugin>
-      </hardware>
-      <joint name="left_hip_joint">
-        <command_interface name="position"/>
-        <state_interface name="position"/>
-        <state_interface name="velocity"/>
-      </joint>
-      <joint name="left_foot_joint">
-        <command_interface name="position"/>
-        <state_interface name="position"/>
-        <state_interface name="velocity"/>
-      </joint>
-      <joint name="right_hip_joint">
-        <command_interface name="position"/>
-        <state_interface name="position"/>
-        <state_interface name="velocity"/>
-      </joint>
-      <joint name="right_foot_joint">
-        <command_interface name="position"/>
-        <state_interface name="position"/>
-        <state_interface name="velocity"/>
-      </joint>
-    </ros2_control>
   </robot>

File: otto_description/urdf/otto_main.urdf.xacro (robot description, xacro)
@@ -1,28 +1,4 @@
 <?xml version="1.0"?>
 <robot xmlns:xacro="http://www.ros.org/wiki/xacro" name="otto">
-  <!-- ============================================================
-       OTTO ROBOT — Main URDF model
-       otto_main.urdf.xacro
-       Kinematic structure
-       ───────────────────
-       base_link  (virtual, at floor level)
-         └── body_link          [fixed]    — torso + head box
-               ├── left_eye     [fixed]    — ultrasonic sensor L  (macro)
-               ├── right_eye    [fixed]    — ultrasonic sensor R  (macro)
-               ├── left_hip_servo  [fixed] — servo block L  (macro)
-               │     └── left_hip_joint   [revolute, Z]
-               │           └── left_leg_link
-               │                 └── left_foot_joint [revolute, Z]
-               │                       └── left_foot_link
-               └── right_hip_servo [fixed] — servo block R  (macro)
-                     └── right_hip_joint  [revolute, Z]
-                           └── right_leg_link
-                                 └── right_foot_joint [revolute, Z]
-                                       └── right_foot_link
-       Coordinate convention
-       ──────────────────────
-       +X  forward   +Y  left   +Z  up
-       All dimensions in metres, masses in kg.
-  ============================================================ -->
   <!-- ── Include utilities ── -->
   <xacro:include filename="otto_materials.xacro" />

Commit message: Working diff_drive not yet operational

File: otto_description/urdf/otto_gz.xacro (robot description, xacro)
@@ -47,4 +47,20 @@
       </visual>
     </gazebo>
+    <!--<gazebo reference="right_back_support_link">
+        <mu1>0</mu1>
+        <mu2>0</mu2>
+    </gazebo>
+     <gazebo reference="right_front_support_link">
+        <mu1>0</mu1>
+        <mu2>0</mu2>
+    </gazebo>
+     <gazebo reference="left_back_support_link">
+        <mu1>0</mu1>
+        <mu2>0</mu2>
+    </gazebo>
+     <gazebo reference="left_front_support_link">
+        <mu1>0</mu1>
+        <mu2>0</mu2>
+    </gazebo>-->
     <!-- Gazebo's Plugins -->
     <gazebo>
@@ -60,4 +76,22 @@
         <joint_name>right_foot_joint</joint_name>
       </plugin>
+      <!-- Differential Drive Plugin -->
+      <plugin filename="gz-sim-diff-drive-system" name="gz::sim::systems::DiffDrive">
+        <!-- Wheels configuration  -->
+        <left_joint>left_foot_joint</left_joint>
+        <right_joint>right_foot_joint</right_joint>
+        <wheel_separations>0.045</wheel_separations>
+        <wheel_radius>0.03</wheel_radius>
+        <!-- output: Control and Odometry (position) -->
+        <odom_publish_frequency>50</odom_publish_frequency>
+        <!-- Input -->
+        <topic>cmd_vel</topic>
+        <!-- Topics Gazebo will publish the data to -->
+      <odom_topic>odom</odom_topic>
+      <tf_topic>tf</tf_topic>
+      <!-- Coordinate frames for RViz and Navigation -->
+      <frame_id>odom</frame_id>
+      <child_frame_id>base_link</child_frame_id>
+      </plugin>
     </gazebo>
   </robot>

File: otto_description/urdf/otto_main.urdf.xacro (robot description, xacro)
@@ -98,5 +98,5 @@
     <parent link="left_hip_servo"/>
     <child  link="left_leg_link"/>
-    <origin xyz="0 0 ${-leg_z/2.0}" rpy="0 0 0"/>
+    <origin xyz="0 0 ${-leg_z/2.0}" rpy="1.5708 0 0"/>
     <axis   xyz="1 0 0"/>
     <limit  lower="${-servo_limit}" upper="${servo_limit}"
@@ -187,5 +187,5 @@
   </link>
   <!-- Foot revolute joint — rotates about Z (tilt foot) -->
-  <joint name="left_foot_joint" type="revolute">
+  <joint name="left_foot_joint" type="continuous">
     <parent link="left_leg_link"/>
     <child  link="left_foot_link"/>
@@ -221,5 +221,5 @@
     <parent link="right_hip_servo"/>
     <child  link="right_leg_link"/>
-    <origin xyz="0 0 ${-leg_z/2.0}" rpy="0 0 0"/>
+    <origin xyz="0 0 ${-leg_z/2.0}" rpy="-1.5708 0 0"/>
     <axis   xyz="1 0 0"/>
     <limit  lower="${-servo_limit}" upper="${servo_limit}"
@@ -308,5 +308,5 @@
     </collision>
   </link>
-  <joint name="right_foot_joint" type="revolute">
+  <joint name="right_foot_joint" type="continuous">
     <parent link="right_leg_link"/>
     <child  link="right_foot_link"/>

Commit message: Rolling ok with issues

File: otto_description/urdf/otto_gz.xacro (robot description, xacro)
@@ -47,5 +47,5 @@
       </visual>
     </gazebo>
-    <!--<gazebo reference="right_back_support_link">
+    <gazebo reference="right_back_support_link">
         <mu1>0</mu1>
         <mu2>0</mu2>
@@ -62,5 +62,5 @@
         <mu1>0</mu1>
         <mu2>0</mu2>
-    </gazebo>-->
+    </gazebo>
     <!-- Gazebo's Plugins -->
     <gazebo>

File: otto_description/urdf/otto_main.urdf.xacro (robot description, xacro)
@@ -13,5 +13,5 @@
   <xacro:property name="leg_x"    value="0.020"/>
   <xacro:property name="leg_y"    value="0.015"/>
-  <xacro:property name="leg_z"    value="0.035"/>
+  <xacro:property name="leg_z"    value="0.018"/>
   <xacro:property name="leg_mass" value="0.025"/>
   <!-- Bar segment -->
@@ -27,5 +27,5 @@
   <!-- Foot (flat disc) -->
   <xacro:property name="foot_r"    value="0.030"/>
-  <xacro:property name="foot_h"    value="0.008"/>
+  <xacro:property name="foot_h"    value="0.005"/>
   <xacro:property name="foot_mass" value="0.020"/>
   <!-- Servo joint limits (±360° realistic for Otto walk) -->

File: otto_description/urdf/otto_materials.xacro (robot description, xacro)
@@ -71,9 +71,9 @@
     <!-- Servo body -->
     <link name="${prefix}_servo">
-      <xacro:inertia_box m="0.009" x="0.023" y="0.012" z="0.045"/>
+      <xacro:inertia_box m="0.009" x="0.023" y="0.012" z="0.03"/>
       <visual>
         <origin xyz="0 0 0" rpy="0 0 0"/>
         <geometry>
-          <box size="0.023 0.012 0.045"/>
+          <box size="0.023 0.012 0.03"/>
         </geometry>
         <material name="otto_dark_grey"/>
@@ -82,5 +82,5 @@
         <origin xyz="0 0 0" rpy="0 0 0"/>
         <geometry>
-          <box size="0.023 0.012 0.045"/>
+          <box size="0.023 0.012 0.03"/>
         </geometry>
       </collision>

Commit message: Setup ros2_control

File: otto_description/urdf/otto_gz.xacro (robot description, xacro)
@@ -1,66 +1,4 @@
 <?xml version="1.0"?>
 <robot xmlns:xacro="http://www.ros.org/wiki/xacro">
-  <!-- GAZEBO PLUGINS -->
-  <!-- Color setting -->
-    <gazebo reference="body_link">
-      <visual>
-        <material>
-          <ambient>0.18 0.52 0.80 1.0</ambient>       <!-- Lighting: dictates what the object looks like when it is in the shadows -->
-          <diffuse>0.18 0.52 0.80 1.0</diffuse>       <!-- Color : object reflects when a direct light source (like the sun or a spotlight) hits it.-->
-        </material>
-      </visual>
-    </gazebo>
-    <gazebo reference="left_leg_link">
-      <visual>
-        <material>
-          <ambient>0.18 0.52 0.80 1.0</ambient>
-          <diffuse>0.18 0.52 0.80 1.0</diffuse>
-        </material>
-      </visual>
-    </gazebo>
-    <gazebo reference="right_leg_link">
-      <visual>
-        <material>
-          <ambient>0.18 0.52 0.80 1.0</ambient>
-          <diffuse>0.18 0.52 0.80 1.0</diffuse>
-        </material>
-      </visual>
-    </gazebo>
-    <gazebo reference="left_foot_link">
-      <mu1>0.9</mu1>
-      <mu2>0.9</mu2>
-      <visual>
-        <material>
-          <ambient>0.65 0.65 0.65 1.0</ambient>
-          <diffuse>0.65 0.65 0.65 1.0</diffuse>
-        </material>
-      </visual>
-    </gazebo>
-    <gazebo reference="right_foot_link">
-      <mu1>0.9</mu1>                              <!-- Friction/gripping on the floor. -->
-      <mu2>0.9</mu2>
-      <visual>
-        <material>
-          <ambient>0.65 0.65 0.65 1.0</ambient>
-          <diffuse>0.65 0.65 0.65 1.0</diffuse>
-        </material>
-      </visual>
-    </gazebo>
-    <gazebo reference="right_back_support_link">
-        <mu1>0</mu1>
-        <mu2>0</mu2>
-    </gazebo>
-     <gazebo reference="right_front_support_link">
-        <mu1>0</mu1>
-        <mu2>0</mu2>
-    </gazebo>
-     <gazebo reference="left_back_support_link">
-        <mu1>0</mu1>
-        <mu2>0</mu2>
-    </gazebo>
-     <gazebo reference="left_front_support_link">
-        <mu1>0</mu1>
-        <mu2>0</mu2>
-    </gazebo>
     <!-- Gazebo's Plugins -->
     <gazebo>

File: otto_description/urdf/otto_main.urdf.xacro (robot description, xacro)
@@ -3,5 +3,5 @@
   <!-- ── Include utilities ── -->
   <xacro:include filename="otto_materials.xacro" />
-  <xacro:include filename="otto_gz.xacro" />
+  <xacro:include filename="otto_ros2_control.xacro" />
   <!--==== PHYSICAL PARAMETERS ====-->
   <!-- Body / head combined box -->

File: otto_description/urdf/otto_materials.xacro (robot description, xacro)
@@ -92,10 +92,5 @@
     </joint>
   </xacro:macro>
-  <!--
-       ULTRASONIC SENSOR MACRO  (HC-SR04 style — the "eyes")
-       parent_link : body/head link
-       side        : "left" | "right"
-       xyz / rpy   : pose in parent frame
-     -->
+  <!-- ULTRASONIC SENSOR MACRO -->
   <xacro:macro name="ultrasonic_eye" params="side parent_link xyz rpy">
     <link name="${side}_eye">
@@ -121,3 +116,64 @@
     </joint>
   </xacro:macro>
+   <!--=========== GAZEBO: Color setting ===========-->
+    <gazebo reference="body_link">
+      <visual>
+        <material>
+          <ambient>0.18 0.52 0.80 1.0</ambient>       <!-- Lighting: dictates what the object looks like when it is in the shadows -->
+          <diffuse>0.18 0.52 0.80 1.0</diffuse>       <!-- Color : object reflects when a direct light source (like the sun or a spotlight) hits it.-->
+        </material>
+      </visual>
+    </gazebo>
+    <gazebo reference="left_leg_link">
+      <visual>
+        <material>
+          <ambient>0.18 0.52 0.80 1.0</ambient>
+          <diffuse>0.18 0.52 0.80 1.0</diffuse>
+        </material>
+      </visual>
+    </gazebo>
+    <gazebo reference="right_leg_link">
+      <visual>
+        <material>
+          <ambient>0.18 0.52 0.80 1.0</ambient>
+          <diffuse>0.18 0.52 0.80 1.0</diffuse>
+        </material>
+      </visual>
+    </gazebo>
+    <gazebo reference="left_foot_link">
+      <mu1>0.9</mu1>
+      <mu2>0.9</mu2>
+      <visual>
+        <material>
+          <ambient>0.65 0.65 0.65 1.0</ambient>
+          <diffuse>0.65 0.65 0.65 1.0</diffuse>
+        </material>
+      </visual>
+    </gazebo>
+    <gazebo reference="right_foot_link">
+      <mu1>0.9</mu1>                               <!--Friction/gripping on the floor.-->
+      <mu2>0.9</mu2>
+      <visual>
+        <material>
+          <ambient>0.65 0.65 0.65 1.0</ambient>
+          <diffuse>0.65 0.65 0.65 1.0</diffuse>
+        </material>
+      </visual>
+    </gazebo>
+    <gazebo reference="right_back_support_link">
+        <mu1>0</mu1>
+        <mu2>0</mu2>
+    </gazebo>
+     <gazebo reference="right_front_support_link">
+        <mu1>0</mu1>
+        <mu2>0</mu2>
+    </gazebo>
+     <gazebo reference="left_back_support_link">
+        <mu1>0</mu1>
+        <mu2>0</mu2>
+    </gazebo>
+     <gazebo reference="left_front_support_link">
+        <mu1>0</mu1>
+        <mu2>0</mu2>
+    </gazebo>
 </robot>
