Commit message: Add sensors(cam & lidar)

File: otto_description/urdf/otto_camera.xacro (robot description, xacro)
@@ -7,5 +7,4 @@
     </joint>
     <link name="camera_link">
-        <xacro:inertia_box m="0.005" x="0.005" y="0.005" z="0.003"/>
         <visual>
             <origin xyz="0 0 0" rpy="0 0 0"/>
@@ -15,4 +14,5 @@
             <material name="otto_black"/>
         </visual>
+        <!--<xacro:inertia_box m="0.005" x="0.005" y="0.005" z="0.003"/>
         <collision>
             <origin xyz="0 0 0" rpy="0 0 0"/>
@@ -20,5 +20,38 @@
                 <box size="0.005 0.005 0.003"/>
             </geometry>
-        </collision>
+        </collision>-->
     </link>
+     <!-- Invisible Joint -->
+    <joint name="camera_optical_joint" type="fixed">
+        <parent link="camera_link"/>
+        <child link="camera_optical_link"/>
+        <origin xyz="0 0 0" rpy="-1.5708 0 -1.5708"/>
+    </joint>
+    <link name="camera_optical_link"></link>
+    <!-- =========== Gazebo tag ========== -->
+    <gazebo reference="camera_link">
+        <sensor name="camera_sensor" type="camera">
+            <always_on>true</always_on>
+            <update_rate>30.0</update_rate>
+            <topic>/camera/image_raw</topic>
+            <gz_frame_id>camera_optical_link</gz_frame_id>
+            <camera>
+                <horizontal_fov>1.39626</horizontal_fov>
+                <image>
+                    <width>640</width>
+                    <height>480</height>
+                    <format>R8G8B8</format>
+                </image>
+                <clip>
+                    <near>0.02</near>
+                    <far>300</far>
+                </clip>
+                <noise>
+                    <type>gaussian</type>
+                    <mean>0.0</mean>
+                    <stddev>0.007</stddev>
+                </noise>
+            </camera>
+        </sensor>
+    </gazebo>
 </robot>

File: otto_description/urdf/otto_lidar.xacro (robot description, xacro)
@@ -22,3 +22,35 @@
         </collision>
     </link>
+    <!-- =========== Gazebo tag ========== -->
+    <gazebo reference="lidar_link">
+        <sensor name="lidar_sensor" type="gpu_lidar">   <!-- Ray: scanning sensor (lidar)-->
+            <always_on>true</always_on>
+            <update_rate>10</update_rate>
+            <topic>/scan</topic>
+            <gz_frame_id>lidar_link</gz_frame_id>
+            <ray>
+                <scan>
+                    <horizontal>
+                        <samples>360</samples>
+                        <resolution>1.0</resolution>
+                        <min_angle>-3.14159</min_angle>
+                        <max_angle>3.14159</max_angle>
+                    </horizontal>
+                </scan>
+                <range>
+                    <min>0.12</min>
+                    <max>8.0</max>
+                    <resolution>0.01</resolution>
+                </range>
+                <noise>
+                    <type>gaussian</type>
+                    <mean>0.0</mean>
+                    <stddev>0.01</stddev>
+                </noise>
+            </ray>
+            <plugin filename="gz-sim-sensors-system" name="gz::sim::systems::Sensors">
+                <render_engine>ogre2</render_engine>
+            </plugin>
+        </sensor>
+    </gazebo>
 </robot>

File: otto_description/urdf/otto_materials.xacro (robot description, xacro)
@@ -119,5 +119,5 @@
     <gazebo reference="left_foot_link">
       <mu1>0.9</mu1>  <!-- forward friction: keep high -->
-      <mu2>0.3</mu2>   <!-- lateral friction: lower to prevent pivot -->
+      <mu2>0.9</mu2>   <!-- lateral friction:  -->
       <visual>
         <material>
@@ -129,5 +129,5 @@
     <gazebo reference="right_foot_link">
       <mu1>0.9</mu1>                               <!--Friction/gripping on the floor.-->
-      <mu2>0.3</mu2>
+      <mu2>0.9</mu2>
       <visual>
         <material>
