Commit message: Add gazebo test

File: otto_description/urdf/otto_main.urdf.xacro (robot description, xacro)
@@ -26,8 +26,6 @@
   ============================================================ -->
   <!-- ── Include utilities ── -->
-  <xacro:include filename="$(find otto_description)/urdf/otto_materials.xacro"/>
-  <!-- ──────────────────────────────────────────────────────────
-       PHYSICAL PARAMETERS  (tweak here to match your print)
-  ────────────────────────────────────────────────────────────── -->
+  <xacro:include filename="otto_materials.xacro" />
+  <!--==== PHYSICAL PARAMETERS ====-->
   <!-- Body / head combined box -->
   <xacro:property name="body_x"    value="0.075"/>   <!-- width  -->
@@ -57,11 +55,7 @@
   <!-- foot joint is at the bottom of the leg -->
   <xacro:property name="foot_z_in_leg"    value="${-leg_z/2.0}"/>
-  <!-- ──────────────────────────────────────────────────────────
-       BASE LINK  (world / floor anchor, mass-less)
-  ────────────────────────────────────────────────────────────── -->
+  <!--=== BASE LINK  (world / floor anchor, mass-less) ===-->
   <link name="base_link"/>
-  <!-- ──────────────────────────────────────────────────────────
-       BODY / HEAD LINK
-  ────────────────────────────────────────────────────────────── -->
+  <!--=== BODY / HEAD LINK ===-->
   <link name="body_link">
     <xacro:inertia_box m="${body_mass}" x="${body_x}" y="${body_y}" z="${body_z}"/>
@@ -94,8 +88,6 @@
     <origin xyz="0 0 ${body_z_from_base}" rpy="0 0 0"/>
   </joint>
-  <!-- ──────────────────────────────────────────────────────────
-       ULTRASONIC EYES  (macro from otto_materials.xacro)
-       Placed on the front face (+X), mirrored on Y axis
-  ────────────────────────────────────────────────────────────── -->
+  <!--=== ULTRASONIC EYES  (macro from otto_materials.xacro)
+       Placed on the front face (+X), mirrored on Y axis  ===-->
   <xacro:ultrasonic_eye
     side="left"
@@ -108,7 +100,5 @@
     xyz="${body_x/2.0 + 0.006} -0.018  ${body_z*0.15}"
     rpy="0 ${pi/2} 0"/>
-  <!-- ──────────────────────────────────────────────────────────
-       LEFT LEG ASSEMBLY
-  ────────────────────────────────────────────────────────────── -->
+  <!--=== LEFT LEG ASSEMBLY ===-->
   <!-- Servo block (cosmetic, fixed to body) -->
   <xacro:servo_block
@@ -169,7 +159,5 @@
     </collision>
   </link>
-  <!-- ──────────────────────────────────────────────────────────
-       RIGHT LEG ASSEMBLY  (mirror of left)
-  ────────────────────────────────────────────────────────────── -->
+  <!-- RIGHT LEG ASSEMBLY  (mirror of left) -->
   <xacro:servo_block
     prefix="right_hip"
@@ -227,36 +215,90 @@
     </collision>
   </link>
-  <!-- ──────────────────────────────────────────────────────────
-       GAZEBO PLUGINS / TAGS  (uncomment if using Gazebo)
-  ────────────────────────────────────────────────────────────── -->
-  <!--
+  <!-- GAZEBO PLUGINS / TAGS -->
   <gazebo reference="body_link">
-    <material>Gazebo/Blue</material>
+    <visual>
+      <material>
+        <ambient>0.18 0.52 0.80 1.0</ambient>
+        <diffuse>0.18 0.52 0.80 1.0</diffuse>
+      </material>
+    </visual>
   </gazebo>
   <gazebo reference="left_leg_link">
-    <material>Gazebo/Blue</material>
+    <visual>
+      <material>
+        <ambient>0.18 0.52 0.80 1.0</ambient>
+        <diffuse>0.18 0.52 0.80 1.0</diffuse>
+      </material>
+    </visual>
   </gazebo>
   <gazebo reference="right_leg_link">
-    <material>Gazebo/Blue</material>
+    <visual>
+      <material>
+        <ambient>0.18 0.52 0.80 1.0</ambient>
+        <diffuse>0.18 0.52 0.80 1.0</diffuse>
+      </material>
+    </visual>
   </gazebo>
   <gazebo reference="left_foot_link">
-    <material>Gazebo/Grey</material>
     <mu1>0.9</mu1>
     <mu2>0.9</mu2>
+    <visual>
+      <material>
+        <ambient>0.65 0.65 0.65 1.0</ambient>
+        <diffuse>0.65 0.65 0.65 1.0</diffuse>
+      </material>
+    </visual>
   </gazebo>
   <gazebo reference="right_foot_link">
-    <material>Gazebo/Grey</material>
     <mu1>0.9</mu1>
     <mu2>0.9</mu2>
-  </gazebo>
+    <visual>
+      <material>
+        <ambient>0.65 0.65 0.65 1.0</ambient>
+        <diffuse>0.65 0.65 0.65 1.0</diffuse>
+      </material>
+    </visual>
+  </gazebo>
+  <!-- Gazebo's Plugins -->
   <gazebo>
-    <plugin name="joint_state_publisher"
-            filename="libgazebo_ros_joint_state_publisher.so">
-      <jointName>
-        left_hip_joint, left_foot_joint,
-        right_hip_joint, right_foot_joint
-      </jointName>
+    <!-- gz-sim-joint-state-publisher-system -->
+    <plugin filename="gz-sim-joint-state-publisher-system"
+            name="gz::sim::systems::JointStatePublisher">
+      <topic>joint_states</topic>
+      <joint_name>left_hip_joint</joint_name>
+      <joint_name>left_foot_joint</joint_name>
+      <joint_name>right_hip_joint</joint_name>
+      <joint_name>right_foot_joint</joint_name>
     </plugin>
-  </gazebo>
-  -->
+    <!-- gz_ros2_control -->
+    <plugin filename="gz_ros2_control-system" name="gz_ros2_control::GazeboSimROS2ControlPlugin">
+      <parameters>$(find otto_description)/config/controllers.yaml</parameters>
+    </plugin>
+  </gazebo>
+  <!-- ROS2_control Specifications -->
+  <ros2_control name="GazeboSimSystem" type="system">
+    <hardware>
+      <plugin>gz_ros2_control/GazeboSimSystem</plugin>
+    </hardware>
+    <joint name="left_hip_joint">
+      <command_interface name="position"/>
+      <state_interface name="position"/>
+      <state_interface name="velocity"/>
+    </joint>
+    <joint name="left_foot_joint">
+      <command_interface name="position"/>
+      <state_interface name="position"/>
+      <state_interface name="velocity"/>
+    </joint>
+    <joint name="right_hip_joint">
+      <command_interface name="position"/>
+      <state_interface name="position"/>
+      <state_interface name="velocity"/>
+    </joint>
+    <joint name="right_foot_joint">
+      <command_interface name="position"/>
+      <state_interface name="position"/>
+      <state_interface name="velocity"/>
+    </joint>
+  </ros2_control>
 </robot>

File: otto_description/urdf/otto_materials.xacro (robot description, xacro)
@@ -5,7 +5,5 @@
        otto_materials.xacro
        ============================================================ -->
-  <!-- ──────────────────────────────────────────────────────────
-       COLORS / MATERIALS
-  ────────────────────────────────────────────────────────────── -->
+  <!--==== COLORS / MATERIALS ====-->
   <material name="otto_blue">
     <color rgba="0.18 0.52 0.80 1.0"/>
@@ -23,8 +21,6 @@
     <color rgba="0.05 0.05 0.05 1.0"/>
   </material>
-  <!-- ──────────────────────────────────────────────────────────
-       INERTIA MACROS  (solid primitives)
-  ────────────────────────────────────────────────────────────── -->
-  <!-- Solid box  m [kg], x/y/z [m] -->
+  <!--==== INERTIA MACROS  (solid primitives) ====-->
+  <!-- Solid box  m [kg], x/y/z [m] (Dimension) -->
   <xacro:macro name="inertia_box" params="m x y z">
     <inertial>
@@ -62,26 +58,23 @@
     </inertial>
   </xacro:macro>
-  <!-- ──────────────────────────────────────────────────────────
-       DEFAULT DYNAMICS MACRO
-       Apply to every revolute joint that drives a servo
-  ────────────────────────────────────────────────────────────── -->
+  <!-- DEFAULT DYNAMICS MACRO: Apply to every revolute joint that drives a servo -->
   <xacro:macro name="servo_dynamics">
     <dynamics damping="0.01" friction="0.001"/>
   </xacro:macro>
-  <!-- ──────────────────────────────────────────────────────────
+  <!--
        SERVO GEOMETRY MACRO
-       Represents a generic SG90/MG90 servo block
+       Represents a generic MG90 servo block
        parent_link : link to which the servo body is attached
-       prefix      : unique name prefix  (e.g. "left_hip")
+       prefix      : unique name prefix  ("left_hip")
        xyz / rpy   : pose in parent frame
-  ────────────────────────────────────────────────────────────── -->
+   -->
   <xacro:macro name="servo_block" params="prefix parent_link xyz rpy">
     <!-- Servo body -->
     <link name="${prefix}_servo">
-      <xacro:inertia_box m="0.009" x="0.023" y="0.012" z="0.025"/>
+      <xacro:inertia_box m="0.009" x="0.023" y="0.012" z="0.032"/>
       <visual>
         <origin xyz="0 0 0" rpy="0 0 0"/>
         <geometry>
-          <box size="0.023 0.012 0.025"/>
+          <box size="0.023 0.012 0.032"/>
         </geometry>
         <material name="otto_dark_grey"/>
@@ -90,5 +83,5 @@
         <origin xyz="0 0 0" rpy="0 0 0"/>
         <geometry>
-          <box size="0.023 0.012 0.025"/>
+          <box size="0.023 0.012 0.032"/>
         </geometry>
       </collision>
@@ -100,10 +93,10 @@
     </joint>
   </xacro:macro>
-  <!-- ──────────────────────────────────────────────────────────
+  <!--
        ULTRASONIC SENSOR MACRO  (HC-SR04 style — the "eyes")
        parent_link : body/head link
        side        : "left" | "right"
        xyz / rpy   : pose in parent frame
-  ────────────────────────────────────────────────────────────── -->
+     -->
   <xacro:macro name="ultrasonic_eye" params="side parent_link xyz rpy">
     <link name="${side}_eye">

Commit message: Add gazebo features

File: otto_description/urdf/otto_main.urdf.xacro (robot description, xacro)
@@ -27,4 +27,5 @@
   <!-- ── Include utilities ── -->
   <xacro:include filename="otto_materials.xacro" />
+  <xacro:include filename="otto_gz.gazebo" />
   <!--==== PHYSICAL PARAMETERS ====-->
   <!-- Body / head combined box -->
@@ -215,90 +216,3 @@
     </collision>
   </link>
-  <!-- GAZEBO PLUGINS / TAGS -->
-  <gazebo reference="body_link">
-    <visual>
-      <material>
-        <ambient>0.18 0.52 0.80 1.0</ambient>
-        <diffuse>0.18 0.52 0.80 1.0</diffuse>
-      </material>
-    </visual>
-  </gazebo>
-  <gazebo reference="left_leg_link">
-    <visual>
-      <material>
-        <ambient>0.18 0.52 0.80 1.0</ambient>
-        <diffuse>0.18 0.52 0.80 1.0</diffuse>
-      </material>
-    </visual>
-  </gazebo>
-  <gazebo reference="right_leg_link">
-    <visual>
-      <material>
-        <ambient>0.18 0.52 0.80 1.0</ambient>
-        <diffuse>0.18 0.52 0.80 1.0</diffuse>
-      </material>
-    </visual>
-  </gazebo>
-  <gazebo reference="left_foot_link">
-    <mu1>0.9</mu1>
-    <mu2>0.9</mu2>
-    <visual>
-      <material>
-        <ambient>0.65 0.65 0.65 1.0</ambient>
-        <diffuse>0.65 0.65 0.65 1.0</diffuse>
-      </material>
-    </visual>
-  </gazebo>
-  <gazebo reference="right_foot_link">
-    <mu1>0.9</mu1>
-    <mu2>0.9</mu2>
-    <visual>
-      <material>
-        <ambient>0.65 0.65 0.65 1.0</ambient>
-        <diffuse>0.65 0.65 0.65 1.0</diffuse>
-      </material>
-    </visual>
-  </gazebo>
-  <!-- Gazebo's Plugins -->
-  <gazebo>
-    <!-- gz-sim-joint-state-publisher-system -->
-    <plugin filename="gz-sim-joint-state-publisher-system"
-            name="gz::sim::systems::JointStatePublisher">
-      <topic>joint_states</topic>
-      <joint_name>left_hip_joint</joint_name>
-      <joint_name>left_foot_joint</joint_name>
-      <joint_name>right_hip_joint</joint_name>
-      <joint_name>right_foot_joint</joint_name>
-    </plugin>
-    <!-- gz_ros2_control -->
-    <plugin filename="gz_ros2_control-system" name="gz_ros2_control::GazeboSimROS2ControlPlugin">
-      <parameters>$(find otto_description)/config/controllers.yaml</parameters>
-    </plugin>
-  </gazebo>
-  <!-- ROS2_control Specifications -->
-  <ros2_control name="GazeboSimSystem" type="system">
-    <hardware>
-      <plugin>gz_ros2_control/GazeboSimSystem</plugin>
-    </hardware>
-    <joint name="left_hip_joint">
-      <command_interface name="position"/>
-      <state_interface name="position"/>
-      <state_interface name="velocity"/>
-    </joint>
-    <joint name="left_foot_joint">
-      <command_interface name="position"/>
-      <state_interface name="position"/>
-      <state_interface name="velocity"/>
-    </joint>
-    <joint name="right_hip_joint">
-      <command_interface name="position"/>
-      <state_interface name="position"/>
-      <state_interface name="velocity"/>
-    </joint>
-    <joint name="right_foot_joint">
-      <command_interface name="position"/>
-      <state_interface name="position"/>
-      <state_interface name="velocity"/>
-    </joint>
-  </ros2_control>
 </robot>

Commit message: Sucess robot walk

File: otto_description/urdf/otto_main.urdf.xacro (robot description, xacro)
@@ -43,6 +43,6 @@
   <xacro:property name="foot_h"    value="0.008"/>
   <xacro:property name="foot_mass" value="0.020"/>
-  <!-- Servo joint limits (±40° realistic for Otto walk) -->
-  <xacro:property name="servo_limit" value="0.78"/>   <!-- rad, ~40° -->
+  <!-- Servo joint limits (±360° realistic for Otto walk) -->
+  <xacro:property name="servo_limit" value="3.14"/>   <!-- rad, ~360° -->
   <xacro:property name="servo_vel"   value="3.14"/>     <!-- rad/s     -->
   <xacro:property name="servo_eff"   value="0.5"/>      <!-- N·m       -->
@@ -108,5 +108,5 @@
     xyz="0 ${leg_offset_y} ${hip_z_in_body}"
     rpy="0 0 0"/>
-  <!-- Hip revolute joint — rotates about Z (swing leg fore/aft) -->
+  <!-- Hip revolute joint — rotates about X (swing leg fore/aft) -->
   <joint name="left_hip_joint" type="revolute">
     <parent link="left_hip_servo"/>
@@ -140,5 +140,5 @@
     <origin xyz="0 0 ${foot_z_in_leg - foot_h/2.0}" rpy="0 0 0"/>
     <axis   xyz="0 0 1"/>
-    <limit  lower="${-servo_limit}" upper="${servo_limit}"
+    <limit  lower="${-servo_limit/2}" upper="${servo_limit/2}"
             effort="${servo_eff}"   velocity="${servo_vel}"/>
     <xacro:servo_dynamics/>
@@ -196,5 +196,5 @@
     <origin xyz="0 0 ${foot_z_in_leg - foot_h/2.0}" rpy="0 0 0"/>
     <axis   xyz="0 0 1"/>
-    <limit  lower="${-servo_limit}" upper="${servo_limit}"
+    <limit  lower="${-servo_limit/2}" upper="${servo_limit/2}"
             effort="${servo_eff}"   velocity="${servo_vel}"/>
     <xacro:servo_dynamics/>

Commit message: Add bracket for rolling stabilization

File: otto_description/urdf/otto_main.urdf.xacro (robot description, xacro)
@@ -39,7 +39,17 @@
   <xacro:property name="leg_z"    value="0.035"/>
   <xacro:property name="leg_mass" value="0.025"/>
+  <!-- Bar segment -->
+  <xacro:property name="bar_x"    value="0.08"/>
+  <xacro:property name="bar_y"    value="0.002"/>
+  <xacro:property name="bar_z"    value="0.0015"/>
+  <xacro:property name="bar_mass" value="0.005"/>
+  <!-- Bar support segment -->
+  <xacro:property name="support_x"    value="0.009"/>
+  <xacro:property name="support_y"    value="0.014"/>
+  <xacro:property name="support_z"    value="0.0015"/>
+  <xacro:property name="support_mass" value="0.001"/>
   <!-- Foot (flat disc) -->
   <xacro:property name="foot_r"    value="0.030"/>
-  <xacro:property name="foot_h"    value="0.008"/>
+  <xacro:property name="foot_h"    value="0.007"/>
   <xacro:property name="foot_mass" value="0.020"/>
   <!-- Servo joint limits (±360° realistic for Otto walk) -->
@@ -134,4 +144,70 @@
     </collision>
   </link>
+  <!-- Balance bar -->
+  <joint name="left_bar_joint" type="fixed">
+    <origin xyz="0.0 ${-leg_y/2} ${-leg_z/2 + bar_z}" rpy="0.0 0.0 0.0"/>
+    <parent link="left_leg_link"/>
+    <child link="left_bar_link"/>
+  </joint>
+  <!-- Left front support -->
+  <joint name="left_front_support_joint" type="fixed">
+    <origin xyz="${bar_x/2 - support_x/2} ${-support_y/2} 0" rpy="0.0 0.0 0.0"/>
+    <parent link="left_bar_link"/>
+    <child link="left_front_support_link"/>
+  </joint>
+   <link name="left_front_support_link">
+    <xacro:inertia_box m="${support_mass}" x="${support_x}" y="${support_y}" z="${support_z}"/>
+    <visual>
+      <origin xyz="0.0 0.0 0.0" rpy="0.0 0.0 0.0"/>
+      <geometry>
+        <box size="${support_x} ${support_y} ${support_z}"/>
+      </geometry>
+      <material name="otto_blue"/>
+    </visual>
+    <collision>
+      <origin xyz="0.0 0.0 0.0" rpy="0.0 0.0 0.0"/>
+      <geometry>
+        <box size="${support_x} ${support_y} ${support_z}"/>
+      </geometry>
+    </collision>
+  </link>
+  <!--Left back support -->
+  <joint name="left_back_support_joint" type="fixed">
+    <origin xyz="${-bar_x/2 + support_x/2} ${-support_y/2} 0" rpy="0.0 0.0 0.0"/>
+    <parent link="left_bar_link"/>
+    <child link="left_back_support_link"/>
+  </joint>
+  <link name="left_back_support_link">
+    <xacro:inertia_box m="${support_mass}" x="${support_x}" y="${support_y}" z="${support_z}"/>
+    <visual>
+      <origin xyz="0.0 0.0 0.0" rpy="0.0 0.0 0.0"/>
+      <geometry>
+        <box size="${support_x} ${support_y} ${support_z}"/>
+      </geometry>
+      <material name="otto_blue"/>
+    </visual>
+    <collision>
+      <origin xyz="0.0 0.0 0.0" rpy="0.0 0.0 0.0"/>
+      <geometry>
+        <box size="${support_x} ${support_y} ${support_z}"/>
+      </geometry>
+    </collision>
+  </link>
+  <link name="left_bar_link">
+    <xacro:inertia_box m="${bar_mass}" x="${bar_x}" y="${bar_y}" z="${bar_z}"/>
+    <visual>
+      <origin xyz="0.0 0.0 0.0" rpy="0.0 0.0 0.0"/>
+      <geometry>
+        <box size="${bar_x} ${bar_y} ${bar_z}"/>
+      </geometry>
+      <material name="otto_blue"/>
+    </visual>
+    <collision>
+      <origin xyz="0.0 0.0 0.0" rpy="0.0 0.0 0.0"/>
+      <geometry>
+        <box size="${bar_x} ${bar_y} ${bar_z}"/>
+      </geometry>
+    </collision>
+  </link>
   <!-- Foot revolute joint — rotates about Z (tilt foot) -->
   <joint name="left_foot_joint" type="revolute">
@@ -191,4 +267,69 @@
     </collision>
   </link>
+  <joint name="right_bar_joint" type="fixed">
+    <origin xyz="0.0 ${leg_y/2} ${-leg_z/2 + bar_z}" rpy="0.0 0.0 0.0"/>
+    <parent link="right_leg_link"/>
+    <child link="right_bar_link"/>
+  </joint>
+  <link name="right_bar_link">
+    <xacro:inertia_box m="${bar_mass}" x="${bar_x}" y="${bar_y}" z="${bar_z}"/>
+    <visual>
+      <origin xyz="0.0 0.0 0.0" rpy="0.0 0.0 0.0"/>
+      <geometry>
+        <box size="${bar_x} ${bar_y} ${bar_z}"/>
+      </geometry>
+      <material name="otto_blue"/>
+    </visual>
+    <collision>
+      <origin xyz="0.0 0.0 0.0" rpy="0.0 0.0 0.0"/>
+      <geometry>
+        <box size="${bar_x} ${bar_y} ${bar_z}"/>
+      </geometry>
+    </collision>
+  </link>
+  <!-- Right front support -->
+  <joint name="right_front_support_joint" type="fixed">
+    <origin xyz="${bar_x/2 - support_x/2} ${support_y/2} 0" rpy="0.0 0.0 0.0"/>
+    <parent link="right_bar_link"/>
+    <child link="right_front_support_link"/>
+  </joint>
+   <link name="right_front_support_link">
+    <xacro:inertia_box m="${support_mass}" x="${support_x}" y="${support_y}" z="${support_z}"/>
+    <visual>
+      <origin xyz="0.0 0.0 0.0" rpy="0.0 0.0 0.0"/>
+      <geometry>
+        <box size="${support_x} ${support_y} ${support_z}"/>
+      </geometry>
+      <material name="otto_blue"/>
+    </visual>
+    <collision>
+      <origin xyz="0.0 0.0 0.0" rpy="0.0 0.0 0.0"/>
+      <geometry>
+        <box size="${support_x} ${support_y} ${support_z}"/>
+      </geometry>
+    </collision>
+  </link>
+  <!-- Right back support -->
+  <joint name="right_back_support_joint" type="fixed">
+    <origin xyz="${-bar_x/2 + support_x/2} ${support_y/2} 0" rpy="0.0 0.0 0.0"/>
+    <parent link="right_bar_link"/>
+    <child link="right_back_support_link"/>
+  </joint>
+  <link name="right_back_support_link">
+    <xacro:inertia_box m="${support_mass}" x="${support_x}" y="${support_y}" z="${support_z}"/>
+    <visual>
+      <origin xyz="0.0 0.0 0.0" rpy="0.0 0.0 0.0"/>
+      <geometry>
+        <box size="${support_x} ${support_y} ${support_z}"/>
+      </geometry>
+      <material name="otto_blue"/>
+    </visual>
+    <collision>
+      <origin xyz="0.0 0.0 0.0" rpy="0.0 0.0 0.0"/>
+      <geometry>
+        <box size="${support_x} ${support_y} ${support_z}"/>
+      </geometry>
+    </collision>
+  </link>
   <joint name="right_foot_joint" type="revolute">
     <parent link="right_leg_link"/>

Commit message: switching works but not rolling

File: otto_description/urdf/otto_main.urdf.xacro (robot description, xacro)
@@ -56,5 +56,5 @@
   <xacro:property name="servo_limit" value="3.14"/>   <!-- rad, ~360° -->
   <xacro:property name="servo_vel"   value="3.14"/>     <!-- rad/s     -->
-  <xacro:property name="servo_eff"   value="0.5"/>      <!-- N·m       -->
+  <xacro:property name="servo_eff"   value="5"/>      <!-- N·m       -->
   <!-- Lateral offset: distance from body centre to each leg -->
   <xacro:property name="leg_offset_y" value="0.025"/>
