Commit message: add stabilization

File: otto_description/urdf/otto_main.urdf.xacro (robot description, xacro)
@@ -39,4 +39,14 @@
   <xacro:property name="leg_z"    value="0.035"/>
   <xacro:property name="leg_mass" value="0.025"/>
+  <!-- Bar segment -->
+  <xacro:property name="bar_x"    value="0.08"/>
+  <xacro:property name="bar_y"    value="0.002"/>
+  <xacro:property name="bar_z"    value="0.0015"/>
+  <xacro:property name="bar_mass" value="0.005"/>
+  <!-- Bar support segment -->
+  <xacro:property name="support_x"    value="0.009"/>
+  <xacro:property name="support_y"    value="0.014"/>
+  <xacro:property name="support_z"    value="0.0015"/>
+  <xacro:property name="support_mass" value="0.001"/>
   <!-- Foot (flat disc) -->
   <xacro:property name="foot_r"    value="0.030"/>
@@ -134,4 +144,70 @@
     </collision>
   </link>
+  <!-- Balance bar -->
+  <joint name="left_bar_joint" type="fixed">
+    <origin xyz="0.0 ${-leg_y/2} ${-leg_z/2 + bar_z}" rpy="0.0 0.0 0.0"/>
+    <parent link="left_leg_link"/>
+    <child link="left_bar_link"/>
+  </joint>
+  <!-- Left front support -->
+  <joint name="left_front_support_joint" type="fixed">
+    <origin xyz="${bar_x/2 - support_x/2} ${-support_y/2} 0" rpy="0.0 0.0 0.0"/>
+    <parent link="left_bar_link"/>
+    <child link="left_front_support_link"/>
+  </joint>
+   <link name="left_front_support_link">
+    <xacro:inertia_box m="${support_mass}" x="${support_x}" y="${support_y}" z="${support_z}"/>
+    <visual>
+      <origin xyz="0.0 0.0 0.0" rpy="0.0 0.0 0.0"/>
+      <geometry>
+        <box size="${support_x} ${support_y} ${support_z}"/>
+      </geometry>
+      <material name="otto_blue"/>
+    </visual>
+    <collision>
+      <origin xyz="0.0 0.0 0.0" rpy="0.0 0.0 0.0"/>
+      <geometry>
+        <box size="${support_x} ${support_y} ${support_z}"/>
+      </geometry>
+    </collision>
+  </link>
+  <!--Left back support -->
+  <joint name="left_back_support_joint" type="fixed">
+    <origin xyz="${-bar_x/2 + support_x/2} ${-support_y/2} 0" rpy="0.0 0.0 0.0"/>
+    <parent link="left_bar_link"/>
+    <child link="left_back_support_link"/>
+  </joint>
+  <link name="left_back_support_link">
+    <xacro:inertia_box m="${support_mass}" x="${support_x}" y="${support_y}" z="${support_z}"/>
+    <visual>
+      <origin xyz="0.0 0.0 0.0" rpy="0.0 0.0 0.0"/>
+      <geometry>
+        <box size="${support_x} ${support_y} ${support_z}"/>
+      </geometry>
+      <material name="otto_blue"/>
+    </visual>
+    <collision>
+      <origin xyz="0.0 0.0 0.0" rpy="0.0 0.0 0.0"/>
+      <geometry>
+        <box size="${support_x} ${support_y} ${support_z}"/>
+      </geometry>
+    </collision>
+  </link>
+  <link name="left_bar_link">
+    <xacro:inertia_box m="${bar_mass}" x="${bar_x}" y="${bar_y}" z="${bar_z}"/>
+    <visual>
+      <origin xyz="0.0 0.0 0.0" rpy="0.0 0.0 0.0"/>
+      <geometry>
+        <box size="${bar_x} ${bar_y} ${bar_z}"/>
+      </geometry>
+      <material name="otto_blue"/>
+    </visual>
+    <collision>
+      <origin xyz="0.0 0.0 0.0" rpy="0.0 0.0 0.0"/>
+      <geometry>
+        <box size="${bar_x} ${bar_y} ${bar_z}"/>
+      </geometry>
+    </collision>
+  </link>
   <!-- Foot revolute joint — rotates about Z (tilt foot) -->
   <joint name="left_foot_joint" type="revolute">
@@ -191,4 +267,69 @@
     </collision>
   </link>
+  <joint name="right_bar_joint" type="fixed">
+    <origin xyz="0.0 ${leg_y/2} ${-leg_z/2 + bar_z}" rpy="0.0 0.0 0.0"/>
+    <parent link="right_leg_link"/>
+    <child link="right_bar_link"/>
+  </joint>
+  <link name="right_bar_link">
+    <xacro:inertia_box m="${bar_mass}" x="${bar_x}" y="${bar_y}" z="${bar_z}"/>
+    <visual>
+      <origin xyz="0.0 0.0 0.0" rpy="0.0 0.0 0.0"/>
+      <geometry>
+        <box size="${bar_x} ${bar_y} ${bar_z}"/>
+      </geometry>
+      <material name="otto_blue"/>
+    </visual>
+    <collision>
+      <origin xyz="0.0 0.0 0.0" rpy="0.0 0.0 0.0"/>
+      <geometry>
+        <box size="${bar_x} ${bar_y} ${bar_z}"/>
+      </geometry>
+    </collision>
+  </link>
+  <!-- Right front support -->
+  <joint name="right_front_support_joint" type="fixed">
+    <origin xyz="${bar_x/2 - support_x/2} ${support_y/2} 0" rpy="0.0 0.0 0.0"/>
+    <parent link="right_bar_link"/>
+    <child link="right_front_support_link"/>
+  </joint>
+   <link name="right_front_support_link">
+    <xacro:inertia_box m="${support_mass}" x="${support_x}" y="${support_y}" z="${support_z}"/>
+    <visual>
+      <origin xyz="0.0 0.0 0.0" rpy="0.0 0.0 0.0"/>
+      <geometry>
+        <box size="${support_x} ${support_y} ${support_z}"/>
+      </geometry>
+      <material name="otto_blue"/>
+    </visual>
+    <collision>
+      <origin xyz="0.0 0.0 0.0" rpy="0.0 0.0 0.0"/>
+      <geometry>
+        <box size="${support_x} ${support_y} ${support_z}"/>
+      </geometry>
+    </collision>
+  </link>
+  <!-- Right back support -->
+  <joint name="right_back_support_joint" type="fixed">
+    <origin xyz="${-bar_x/2 + support_x/2} ${support_y/2} 0" rpy="0.0 0.0 0.0"/>
+    <parent link="right_bar_link"/>
+    <child link="right_back_support_link"/>
+  </joint>
+  <link name="right_back_support_link">
+    <xacro:inertia_box m="${support_mass}" x="${support_x}" y="${support_y}" z="${support_z}"/>
+    <visual>
+      <origin xyz="0.0 0.0 0.0" rpy="0.0 0.0 0.0"/>
+      <geometry>
+        <box size="${support_x} ${support_y} ${support_z}"/>
+      </geometry>
+      <material name="otto_blue"/>
+    </visual>
+    <collision>
+      <origin xyz="0.0 0.0 0.0" rpy="0.0 0.0 0.0"/>
+      <geometry>
+        <box size="${support_x} ${support_y} ${support_z}"/>
+      </geometry>
+    </collision>
+  </link>
   <joint name="right_foot_joint" type="revolute">
     <parent link="right_leg_link"/>

Commit message: Test walking mode - validate

File: otto_description/urdf/otto_main.urdf.xacro (robot description, xacro)
@@ -98,5 +98,5 @@
     <parent link="left_hip_servo"/>
     <child  link="left_leg_link"/>
-    <origin xyz="0 0 ${-leg_z/2.0}" rpy="1.5708 0 0"/>
+    <origin xyz="0 0 ${-leg_z/2.0}" rpy="0 0 0"/>
     <axis   xyz="1 0 0"/>
     <limit  lower="${-servo_limit}" upper="${servo_limit}"
@@ -221,5 +221,5 @@
     <parent link="right_hip_servo"/>
     <child  link="right_leg_link"/>
-    <origin xyz="0 0 ${-leg_z/2.0}" rpy="-1.5708 0 0"/>
+    <origin xyz="0 0 ${-leg_z/2.0}" rpy="0 0 0"/>
     <axis   xyz="1 0 0"/>
     <limit  lower="${-servo_limit}" upper="${servo_limit}"

File: otto_description/urdf/otto_ros2_control.xacro (robot description, xacro)
@@ -11,8 +11,5 @@
         <joint name="left_foot_joint">
             <!-- Data to send -->
-            <command_interface name="velocity">
-                <param name="min">-10</param>
-                <param name="max">10</param>
-            </command_interface>
+            <command_interface name="position"/>
             <!-- Data to read only -->
             <state_interface name="velocity"/>
@@ -20,8 +17,5 @@
         </joint>
         <joint name="right_foot_joint">
-            <command_interface name="velocity">
-                <param name="min">-10</param>
-                <param name="max">10</param>
-            </command_interface>
+            <command_interface name="position"/>
             <state_interface name="velocity"/>
             <state_interface name="position"/>

Commit message: Added sensors

File: otto_description/urdf/otto_main.urdf.xacro (robot description, xacro)
@@ -4,4 +4,7 @@
   <xacro:include filename="otto_materials.xacro" />
   <xacro:include filename="otto_ros2_control.xacro" />
+  <xacro:include filename="otto_lidar.xacro" />
+  <xacro:include filename="otto_camera.xacro" />
+  <xacro:include filename="otto_display.xacro" />
   <!--==== PHYSICAL PARAMETERS ====-->
   <!-- Body / head combined box -->
@@ -75,16 +78,4 @@
     <origin xyz="0 0 ${body_z_from_base}" rpy="0 0 0"/>
   </joint>
-  <!--=== ULTRASONIC EYES  (macro from otto_materials.xacro)
-       Placed on the front face (+X), mirrored on Y axis  ===-->
-  <xacro:ultrasonic_eye
-    side="left"
-    parent_link="body_link"
-    xyz="${body_x/2.0 + 0.006}  0.018  ${body_z*0.15}"
-    rpy="0 ${pi/2} 0"/>
-  <xacro:ultrasonic_eye
-    side="right"
-    parent_link="body_link"
-    xyz="${body_x/2.0 + 0.006} -0.018  ${body_z*0.15}"
-    rpy="0 ${pi/2} 0"/>
   <!--=== LEFT LEG ASSEMBLY ===-->
   <!-- Servo block (cosmetic, fixed to body) -->

File: otto_description/urdf/otto_materials.xacro (robot description, xacro)
@@ -92,28 +92,4 @@
     </joint>
   </xacro:macro>
-  <!-- ULTRASONIC SENSOR MACRO -->
-  <xacro:macro name="ultrasonic_eye" params="side parent_link xyz rpy">
-    <link name="${side}_eye">
-      <xacro:inertia_cylinder m="0.003" r="0.008" h="0.012"/>
-      <visual>
-        <origin xyz="0 0 0" rpy="0 0 0"/>
-        <geometry>
-          <cylinder radius="0.008" length="0.012"/>
-        </geometry>
-        <material name="otto_black"/>
-      </visual>
-      <collision>
-        <origin xyz="0 0 0" rpy="0 0 0"/>
-        <geometry>
-          <cylinder radius="0.008" length="0.012"/>
-        </geometry>
-      </collision>
-    </link>
-    <joint name="${side}_eye_joint" type="fixed">
-      <parent link="${parent_link}"/>
-      <child  link="${side}_eye"/>
-      <origin xyz="${xyz}" rpy="${rpy}"/>
-    </joint>
-  </xacro:macro>
    <!--=========== GAZEBO: Color setting ===========-->
     <gazebo reference="body_link">

Commit message: Start fixing axis issue

File: otto_description/urdf/otto_main.urdf.xacro (robot description, xacro)
@@ -78,4 +78,11 @@
     <origin xyz="0 0 ${body_z_from_base}" rpy="0 0 0"/>
   </joint>
+  <!-- Base footprint -->
+  <link name="base_footprint"/>
+  <joint name="base_footprint_joint" type="fixed">
+      <parent link="base_footprint"/>
+      <child link="base_link"/>
+      <origin xyz="0 0 0.10" rpy="0 0 0"/>
+  </joint>
   <!--=== LEFT LEG ASSEMBLY ===-->
   <!-- Servo block (cosmetic, fixed to body) -->
@@ -178,5 +185,5 @@
   </link>
   <!-- Foot revolute joint — rotates about Z (tilt foot) -->
-  <joint name="left_foot_joint" type="continuous">
+  <joint name="left_foot_joint" type="revolute">
     <parent link="left_leg_link"/>
     <child  link="left_foot_link"/>
@@ -189,13 +196,29 @@
   <link name="left_foot_link">
     <xacro:inertia_cylinder m="${foot_mass}" r="${foot_r}" h="${foot_h}"/>
-    <visual>
-      <origin xyz="0 0 0" rpy="0 0 0"/>
-      <geometry>
-        <cylinder radius="${foot_r}" length="${foot_h}"/>
-      </geometry>
-      <material name="otto_grey"/>
-    </visual>
-    <collision>
-      <origin xyz="0 0 0" rpy="0 0 0"/>
+    <collision>
+      <origin xyz="0 0 0" rpy="0 0 0"/>
+      <geometry>
+        <cylinder radius="${foot_r}" length="${foot_h}"/>
+      </geometry>
+    </collision>
+  </link>
+  <joint name="left_wheel_joint" type="continuous">
+    <parent link="left_foot_link"/>
+    <child  link="left_wheel_link"/>
+    <origin xyz="0 0 -0.01" rpy="0 0 0"/> <axis   xyz="0 0 1"/> </joint>
+  <link name="left_wheel_link">
+      <inertial>
+      <mass value="0.01"/>
+      <inertia ixx="0.00001" ixy="0" ixz="0" iyy="0.00001" iyz="0" izz="0.00001"/>
+    </inertial>
+    <visual>
+      <origin xyz="0 0 0" rpy="1.5708 0 0"/>
+      <geometry>
+        <cylinder radius="${foot_r}" length="${foot_h}"/>
+      </geometry>
+      <material name="otto_black"/>
+    </visual>
+    <collision>
+      <origin xyz="0 0 0" rpy="1.5708 0 0"/>
       <geometry>
         <cylinder radius="${foot_r}" length="${foot_h}"/>
@@ -299,5 +322,5 @@
     </collision>
   </link>
-  <joint name="right_foot_joint" type="continuous">
+  <joint name="right_foot_joint" type="revolute">
     <parent link="right_leg_link"/>
     <child  link="right_foot_link"/>
@@ -324,3 +347,19 @@
     </collision>
   </link>
+   <joint name="right_wheel_joint" type="continuous">
+    <parent link="right_foot_link"/>
+    <child  link="right_wheel_link"/>
+    <origin xyz="0 0 -0.01" rpy="0 0 0"/> <axis   xyz="0 0 1"/> </joint>
+  <link name="right_wheel_link">
+     <inertial>
+      <mass value="0.01"/>
+      <inertia ixx="0.00001" ixy="0" ixz="0" iyy="0.00001" iyz="0" izz="0.00001"/>
+    </inertial>
+    <collision>
+      <origin xyz="0 0 0" rpy="1.5708 0 0"/>
+      <geometry>
+        <cylinder radius="${foot_r}" length="${foot_h}"/>
+      </geometry>
+    </collision>
+  </link>
 </robot>

File: otto_description/urdf/otto_ros2_control.xacro (robot description, xacro)
@@ -9,5 +9,5 @@
         <!--== Actuators definition (Joints) ==-->
         <!-- Drive Wheels (Velocity ctrl)-->
-        <joint name="left_foot_joint">
+          <joint name="left_wheel_joint">
             <!-- Data to send -->
             <command_interface name="velocity"/>
@@ -17,5 +17,5 @@
             <state_interface name="position"/>
         </joint>
-        <joint name="right_foot_joint">
+        <joint name="right_wheel_joint">
             <command_interface name="velocity"/>
             <command_interface name="position"/>
@@ -23,5 +23,15 @@
             <state_interface name="position"/>
         </joint>
-        <!-- Bending knees (Position ctrl)-->
+         <!-- Bending knees (Position ctrl)-->
+        <joint name="left_foot_joint">
+            <command_interface name="position"/>
+            <state_interface name="velocity"/>
+            <state_interface name="position"/>
+        </joint>
+        <joint name="right_foot_joint">
+            <command_interface name="position"/>
+            <state_interface name="velocity"/>
+            <state_interface name="position"/>
+        </joint>
         <joint name="left_hip_joint">
             <command_interface name="position"/>

Commit message: Reset

File: otto_description/urdf/otto_main.urdf.xacro (robot description, xacro)
@@ -185,5 +185,5 @@
   </link>
   <!-- Foot revolute joint — rotates about Z (tilt foot) -->
-  <joint name="left_foot_joint" type="revolute">
+  <joint name="left_foot_joint" type="continuous">
     <parent link="left_leg_link"/>
     <child  link="left_foot_link"/>
@@ -196,29 +196,13 @@
   <link name="left_foot_link">
     <xacro:inertia_cylinder m="${foot_mass}" r="${foot_r}" h="${foot_h}"/>
-    <collision>
+     <visual>
       <origin xyz="0 0 0" rpy="0 0 0"/>
       <geometry>
         <cylinder radius="${foot_r}" length="${foot_h}"/>
       </geometry>
-    </collision>
-  </link>
-  <joint name="left_wheel_joint" type="continuous">
-    <parent link="left_foot_link"/>
-    <child  link="left_wheel_link"/>
-    <origin xyz="0 0 -0.01" rpy="0 0 0"/> <axis   xyz="0 0 1"/> </joint>
-  <link name="left_wheel_link">
-      <inertial>
-      <mass value="0.01"/>
-      <inertia ixx="0.00001" ixy="0" ixz="0" iyy="0.00001" iyz="0" izz="0.00001"/>
-    </inertial>
-    <visual>
-      <origin xyz="0 0 0" rpy="1.5708 0 0"/>
-      <geometry>
-        <cylinder radius="${foot_r}" length="${foot_h}"/>
-      </geometry>
-      <material name="otto_black"/>
-    </visual>
-    <collision>
-      <origin xyz="0 0 0" rpy="1.5708 0 0"/>
+      <material name="otto_grey"/>
+    </visual>
+    <collision>
+      <origin xyz="0 0 0" rpy="0 0 0"/>
       <geometry>
         <cylinder radius="${foot_r}" length="${foot_h}"/>
@@ -322,5 +306,5 @@
     </collision>
   </link>
-  <joint name="right_foot_joint" type="revolute">
+  <joint name="right_foot_joint" type="continuous">
     <parent link="right_leg_link"/>
     <child  link="right_foot_link"/>
@@ -347,19 +331,3 @@
     </collision>
   </link>
-   <joint name="right_wheel_joint" type="continuous">
-    <parent link="right_foot_link"/>
-    <child  link="right_wheel_link"/>
-    <origin xyz="0 0 -0.01" rpy="0 0 0"/> <axis   xyz="0 0 1"/> </joint>
-  <link name="right_wheel_link">
-     <inertial>
-      <mass value="0.01"/>
-      <inertia ixx="0.00001" ixy="0" ixz="0" iyy="0.00001" iyz="0" izz="0.00001"/>
-    </inertial>
-    <collision>
-      <origin xyz="0 0 0" rpy="1.5708 0 0"/>
-      <geometry>
-        <cylinder radius="${foot_r}" length="${foot_h}"/>
-      </geometry>
-    </collision>
-  </link>
 </robot>

File: otto_description/urdf/otto_ros2_control.xacro (robot description, xacro)
@@ -8,14 +8,6 @@
         </hardware>
         <!--== Actuators definition (Joints) ==-->
-        <!-- Drive Wheels (Velocity ctrl)-->
-          <joint name="left_wheel_joint">
-            <!-- Data to send -->
-            <command_interface name="velocity"/>
-            <command_interface name="position"/>
-            <!-- Data to read only -->
-            <state_interface name="velocity"/>
-            <state_interface name="position"/>
-        </joint>
-        <joint name="right_wheel_joint">
+         <!-- Bending knees (Position ctrl)-->
+        <joint name="left_foot_joint">
             <command_interface name="velocity"/>
             <command_interface name="position"/>
@@ -23,11 +15,6 @@
             <state_interface name="position"/>
         </joint>
-         <!-- Bending knees (Position ctrl)-->
-        <joint name="left_foot_joint">
-            <command_interface name="position"/>
-            <state_interface name="velocity"/>
-            <state_interface name="position"/>
-        </joint>
         <joint name="right_foot_joint">
+            <command_interface name="velocity"/>
             <command_interface name="position"/>
             <state_interface name="velocity"/>

Commit message: Fixed coordonates switching issues

File: otto_description/urdf/otto_main.urdf.xacro (robot description, xacro)
@@ -185,5 +185,5 @@
   </link>
   <!-- Foot revolute joint — rotates about Z (tilt foot) -->
-  <joint name="left_foot_joint" type="continuous">
+  <joint name="left_foot_joint" type="revolute">
     <parent link="left_leg_link"/>
     <child  link="left_foot_link"/>
@@ -203,4 +203,20 @@
       <material name="otto_grey"/>
     </visual>
+    <collision>
+      <origin xyz="0 0 0" rpy="0 0 0"/>
+      <geometry>
+        <cylinder radius="${foot_r}" length="${foot_h}"/>
+      </geometry>
+    </collision>
+  </link>
+  <joint name="left_wheel_joint" type="continuous">
+    <parent link="left_foot_link"/>
+    <child  link="left_wheel_link"/>
+    <origin xyz="0 0 0" rpy="0 0 0"/> <axis   xyz="0 0 -1"/> </joint>
+ <link name="left_wheel_link">
+    <inertial>
+      <mass value="0.01"/>
+      <inertia ixx="0.00001" ixy="0" ixz="0" iyy="0.00001" iyz="0" izz="0.00001"/>
+    </inertial>
     <collision>
       <origin xyz="0 0 0" rpy="0 0 0"/>
@@ -306,5 +322,5 @@
     </collision>
   </link>
-  <joint name="right_foot_joint" type="continuous">
+  <joint name="right_foot_joint" type="revolute">
     <parent link="right_leg_link"/>
     <child  link="right_foot_link"/>
@@ -331,3 +347,19 @@
     </collision>
   </link>
+   <joint name="right_wheel_joint" type="continuous">
+    <parent link="right_foot_link"/>
+    <child  link="right_wheel_link"/>
+    <origin xyz="0 0 0" rpy="0 0 0"/> <axis   xyz="0 0 1"/> </joint>
+  <link name="right_wheel_link">
+    <inertial>
+      <mass value="0.01"/>
+      <inertia ixx="0.00001" ixy="0" ixz="0" iyy="0.00001" iyz="0" izz="0.00001"/>
+    </inertial>
+    <collision>
+      <origin xyz="0 0 0" rpy="0 0 0"/>
+      <geometry>
+        <cylinder radius="${foot_r}" length="${foot_h}"/>
+      </geometry>
+    </collision>
+  </link>
 </robot>

File: otto_description/urdf/otto_ros2_control.xacro (robot description, xacro)
@@ -8,6 +8,14 @@
         </hardware>
         <!--== Actuators definition (Joints) ==-->
-         <!-- Bending knees (Position ctrl)-->
-        <joint name="left_foot_joint">
+        <!-- Drive Wheels (Velocity ctrl)-->
+          <joint name="left_wheel_joint">
+            <!-- Data to send -->
+            <command_interface name="velocity"/>
+            <command_interface name="position"/>
+            <!-- Data to read only -->
+            <state_interface name="velocity"/>
+            <state_interface name="position"/>
+        </joint>
+        <joint name="right_wheel_joint">
             <command_interface name="velocity"/>
             <command_interface name="position"/>
@@ -15,6 +23,11 @@
             <state_interface name="position"/>
         </joint>
+         <!-- Bending knees (Position ctrl)-->
+        <joint name="left_foot_joint">
+            <command_interface name="position"/>
+            <state_interface name="velocity"/>
+            <state_interface name="position"/>
+        </joint>
         <joint name="right_foot_joint">
-            <command_interface name="velocity"/>
             <command_interface name="position"/>
             <state_interface name="velocity"/>

Commit message: Start checking and upgrade

File: otto_description/urdf/otto_main.urdf.xacro (robot description, xacro)
@@ -12,5 +12,5 @@
   <xacro:property name="body_y"    value="0.060"/>   <!-- depth  -->
   <xacro:property name="body_z"    value="0.065"/>   <!-- height -->
-  <xacro:property name="body_mass" value="0.120"/>
+  <xacro:property name="body_mass" value="0.07"/>
   <!-- Leg segment -->
   <xacro:property name="leg_x"    value="0.020"/>

File: otto_description/urdf/otto_materials.xacro (robot description, xacro)
@@ -118,5 +118,5 @@
     </gazebo>
     <gazebo reference="left_foot_link">
-      <mu1>0.9</mu1>  <!-- forward friction -->
+      <mu1>0.0</mu1>  <!-- forward friction -->
       <mu2>0.9</mu2>   <!-- lateral friction:  -->
       <visual>
@@ -128,5 +128,5 @@
     </gazebo>
     <gazebo reference="right_foot_link">
-      <mu1>0.9</mu1>                               <!--Friction/gripping on the floor.-->
+      <mu1>0.0</mu1>                               <!--Friction/gripping on the floor.-->
       <mu2>0.9</mu2>
       <visual>
